Commit message: Initial version of the project with all parts integrated

File: gazebo_differential_drive_robot/model/robot.xacro (robot description, xacro)
@@ -1,10 +1,9 @@
 <?xml version="1.0"?>
 <robot name="differential_drive_robot" xmlns:xacro="http://www.ros.org/wiki/xacro">
-    <!-- Robot Parameters -->
     <xacro:property name="PI" value="3.14159265"/>
     <xacro:property name="body_length" value="0.5"/>
     <xacro:property name="body_width" value="0.3"/>
     <xacro:property name="body_height" value="0.1"/>
-    <xacro:property name="body_density" value="7850.0"/> <!-- Steel -->
+    <xacro:property name="body_density" value="7850.0"/>
     <xacro:property name="body_mass" value="${body_density * body_length * body_height * body_width}"/>
     <xacro:property name="body_inertia_x" value="${1.0/12.0 * body_mass * (body_height*body_height + body_width*body_width)}"/>
@@ -15,5 +14,5 @@
     <xacro:property name="wheel_separation" value="${body_width + wheel_width}"/>
     <xacro:property name="wheel_offset" value="${body_length/2 - wheel_radius}"/>
-    <xacro:property name="wheel_density" value="900"/> <!-- Ruber -->
+    <xacro:property name="wheel_density" value="900"/>
     <xacro:property name="wheel_mass" value="${wheel_density * PI * wheel_radius * wheel_radius * wheel_width}"/>
     <xacro:property name="wheel_inertia_x" value="${1.0/12.0 * wheel_mass * (3*wheel_radius*wheel_radius + wheel_width*wheel_width)}"/>
@@ -27,8 +26,17 @@
     <xacro:property name="caster_inertia_y" value="${2.0/5.0 * caster_mass * caster_radius * caster_radius}"/>
     <xacro:property name="caster_inertia_z" value="${2.0/5.0 * caster_mass * caster_radius * caster_radius}"/>
-    <!-- Control Parameters -->
     <xacro:property name="max_linear_acceleration" value="10"/>
-    <!-- Links -->
-    <!-- Body Link -->
+    <link name="base_footprint"/>
+    <link name="base_link"/>
+    <joint name="footprint_to_link" type="fixed">
+        <parent link="base_footprint"/>
+        <child link="base_link"/>
+        <origin xyz="0 0 0" rpy="0 0 0"/>
+    </joint>
+    <joint name="base_joint" type="fixed">
+        <parent link="base_link"/>
+        <child link="body_link"/>
+        <origin xyz="0 0 0" rpy="0 0 0"/>
+    </joint>
     <link name="body_link">
         <visual>
@@ -53,5 +61,4 @@
         </inertial>
     </link>
-    <!-- Left Wheel -->
     <link name="left_wheel_link">
         <visual>
@@ -76,5 +83,4 @@
         </inertial>
     </link>
-    <!-- Right Wheel -->
     <link name="right_wheel_link">
         <visual>
@@ -99,5 +105,4 @@
         </inertial>
     </link>
-    <!-- Caster Wheel -->
     <link name="caster_link">
         <visual>
@@ -122,6 +127,26 @@
         </inertial>
     </link>
-    <!-- Joints -->
-    <!-- Left Wheel Joint -->
+    <link name="laser_link">
+        <visual>
+            <origin xyz="0 0 0" rpy="0 0 0"/>
+            <geometry>
+                <cylinder radius="0.05" length="0.04"/>
+            </geometry>
+            <material name="laser_material">
+                <color rgba="1.0 0.0 0.0 1.0"/>
+            </material>
+        </visual>
+        <collision>
+            <origin xyz="0 0 0" rpy="0 0 0"/>
+            <geometry>
+                <cylinder radius="0.05" length="0.04"/>
+            </geometry>
+        </collision>
+        <inertial>
+            <mass value="0.1"/>
+            <inertia ixx="0.0001" ixy="0" ixz="0" iyy="0.0001" iyz="0" izz="0.0001"/>
+            <origin xyz="0 0 0" rpy="0 0 0"/>
+        </inertial>
+    </link>
     <joint name="left_wheel_joint" type="continuous">
         <origin xyz="-${wheel_offset} ${wheel_separation/2} -${wheel_radius/2}" rpy="0 0 0"/>
@@ -132,5 +157,4 @@
         <dynamics damping="0.1" friction="0.1"/>
     </joint>
-    <!-- Right Wheel Joint -->
     <joint name="right_wheel_joint" type="continuous">
         <origin xyz="-${wheel_offset} ${-wheel_separation/2} -${wheel_radius/2}" rpy="0 0 0"/>
@@ -141,5 +165,4 @@
         <dynamics damping="0.1" friction="0.1"/>
     </joint>
-    <!-- Caster Wheel Joint (fixed) -->
     <joint name="caster_joint" type="fixed">
         <origin xyz="${caster_offset} 0 -${caster_radius/2}" rpy="0 0 0"/>
@@ -147,22 +170,70 @@
         <child link="caster_link"/>
     </joint>
-    <!-- Gazebo Parameters -->
+    <joint name="laser_joint" type="fixed">
+        <origin xyz="0 0 ${body_height/2 + 0.02}" rpy="0 0 0"/>
+        <parent link="body_link"/>
+        <child link="laser_link"/>
+    </joint>
     <gazebo reference="body_link">
         <mu1>1.0</mu1>
         <mu2>1.0</mu2>
+        <material>
+            <ambient>0.25 0.25 0.25 1.0</ambient>
+            <diffuse>0.25 0.25 0.25 1.0</diffuse>
+        </material>
     </gazebo>
     <gazebo reference="right_wheel_link">
         <mu1>1.0</mu1>
         <mu2>1.0</mu2>
+        <material>
+            <ambient>0.0 0.0 0.0 1.0</ambient>
+            <diffuse>0.0 0.0 0.0 1.0</diffuse>
+        </material>
     </gazebo>
     <gazebo reference="left_wheel_link">
         <mu1>1.0</mu1>
         <mu2>1.0</mu2>
+        <material>
+            <ambient>0.0 0.0 0.0 1.0</ambient>
+            <diffuse>0.0 0.0 0.0 1.0</diffuse>
+        </material>
     </gazebo>
     <gazebo reference="caster_link">
         <mu1>0.000001</mu1>
         <mu2>0.000001</mu2>
-    </gazebo>
-    <!-- Gazebo Plugins -->
+        <material>
+            <ambient>0.0 0.0 0.0 1.0</ambient>
+            <diffuse>0.0 0.0 0.0 1.0</diffuse>
+        </material>
+    </gazebo>
+    <gazebo reference="laser_link">
+        <material>
+            <ambient>1.0 0.0 0.0 1.0</ambient>
+            <diffuse>1.0 0.0 0.0 1.0</diffuse>
+        </material>
+        <sensor name="lidar" type="gpu_lidar">
+            <pose>0 0 0 0 0 0</pose>
+            <topic>/scan</topic>
+            <gz_frame_id>laser_link</gz_frame_id>
+            <update_rate>10</update_rate>
+            <ray>
+                <scan>
+                    <horizontal>
+                        <samples>360</samples>
+                        <resolution>1</resolution>
+                        <min_angle>-3.14159</min_angle>
+                        <max_angle>3.14159</max_angle>
+                    </horizontal>
+                </scan>
+                <range>
+                    <min>0.12</min>
+                    <max>10.0</max>
+                    <resolution>0.01</resolution>
+                </range>
+            </ray>
+            <always_on>true</always_on>
+            <visualize>true</visualize>
+        </sensor>
+    </gazebo>
     <gazebo>
         <plugin filename="gz-sim-diff-drive-system" name="gz::sim::systems::DiffDrive">
@@ -173,6 +244,9 @@
             <max_linear_acceleration>${max_linear_acceleration}</max_linear_acceleration>
             <odom_publish_frequency>100</odom_publish_frequency>
-            <topic>cmd_vel</topic>
-            <odom_topic>odom</odom_topic>
+            <topic>/cmd_vel</topic>
+            <odom_topic>/odom</odom_topic>
+            <frame_id>odom</frame_id>
+            <child_frame_id>base_footprint</child_frame_id>
+            <tf_topic>/tf</tf_topic>
         </plugin>
         <plugin filename="gz-sim-joint-state-publisher-system" name="gz::sim::systems::JointStatePublisher">
@@ -181,4 +255,7 @@
             <joint_name>left_wheel_joint</joint_name>
         </plugin>
+        <plugin filename="gz-sim-sensors-system" name="gz::sim::systems::Sensors">
+            <render_engine>ogre2</render_engine>
+        </plugin>
     </gazebo>
 </robot>
